File: Electronic Design/SAO Demo Controller V3 Design Files KiCAD 10/SAO_Demo_Controller.kicad_sch (KiCad schematic)
At the start: 56 parts, among them J1 BATT., J2 BATT., SW3 SK12D07L4B, U1 RY2201, U2 TP4054, U3 TPS63070RNMR, U4 NID5100, U5 INA180A2, U6 RP2040-Zero, X1 SAO_conn, X2 SAO_conn, X3 SAO_conn, X5 QWIIC

Commit message: Add special LiPo dedicated use note to schematic
Other:
- note added: "0.3A, 0.30V Drop 0.5A, 0.35V Drop 1.0A, 0.45V Drop"
- note added: "FOR DEDICATED LIPO ONLY USE If you want to only use the 1S LiPo and USB power options (likely for Etch sAO Sketch or similar SAOs) remove ALL diodes D1-4. Solder bridge only the D3 position footpring. These changes will safely provide more runtime and full use of the LiPo capacity. USB Power will still provide direct power to the RP2040-Zero, and power to the Main Switch via the LiPo charging IC."
- note removed: "0.3A, 0.___V 0.5A, 0.___V 1.0A, 0.450V"
Changed lines of the file:
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@@
+		)
+	)
+	(text "FOR DEDICATED LIPO ONLY USE\n\nIf you want to only use the 1S LiPo and USB\npower options (likely for Etch sAO Sketch\nor similar SAOs) remove ALL diodes D1-4.\n\nSolder bridge only the D3 position footpring.\nThese changes will safely provide more runtime\nand full use of the LiPo capacity.\n\nUSB Power will still provide direct power to\nthe RP2040-Zero, and power to the Main Switch\nvia the LiPo charging IC."
+		(exclude_from_sim no)
+		(at 14.224 163.068 0)
+		(effects
+			(font
+				(size 1.27 1.27)
+				(thickness 0.254)
+				(bold yes)
+				(color 255 2 6 1)
+			)
+			(justify left)
 		)
 	)
@@
 		)
 	)
-	(text "0.3A, 0.___V\n0.5A, 0.___V\n1.0A, 0.450V"
+	(text "0.3A, 0.30V Drop\n0.5A, 0.35V Drop\n1.0A, 0.45V Drop"
 		(exclude_from_sim no)
-		(at 195.326 34.036 0)
+		(at 191.77 33.782 0)
 		(effects
 			(font

Commit message: Correct V3 schematic PDF JP4 and 5 text
Other:
- note added: "JP4: SAO GPIO1 Select 1-2 is RP2040 GP1 or SAO in 2-3 is RP2040 GP26/ADC0"
- note added: "JP5: SAO GPIO2 Select 1-2 is RP2040 GP0 or SAO in 2-3 is RP2040 GP27/ADC1"
- note added: "SAO Core4 V2 requires JP5:2-3 closed to use GP27 as input for core pulse sense."
- note removed: "JP5: SAO GPIO1 Select 1-2 is RP2040 GP1 or SAO in 2-3 is RP2040 GP26/ADC0"
- note removed: "JP6: SAO GPIO2 Select 1-2 is RP2040 GP0 or SAO in 2-3 is RP2040 GP27/ADC1"
Changed lines of the file:
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@@
 	(title_block
 		(title "SAO Demo Controller, Micro Badge Development Board")
-		(date "2026-08-15")
+		(date "2026-08-26")
 		(rev "3.0, 3.1, 3.2")
 		(company "Design by Andy Geppert @ www.MachineIdeas.com")
@@
 		)
 	)
-	(text "JP5: SAO GPIO1 Select\n1-2 is RP2040 GP1 or SAO in\n2-3 is RP2040 GP26/ADC0"
+	(text "JP4: SAO GPIO1 Select\n1-2 is RP2040 GP1 or SAO in\n2-3 is RP2040 GP26/ADC0"
 		(exclude_from_sim no)
 		(at 255.524 132.842 0)
@@
 		)
 	)
-	(text "JP6: SAO GPIO2 Select\n1-2 is RP2040 GP0 or SAO in\n2-3 is RP2040 GP27/ADC1"
+	(text "JP5: SAO GPIO2 Select\n1-2 is RP2040 GP0 or SAO in\n2-3 is RP2040 GP27/ADC1"
 		(exclude_from_sim no)
 		(at 255.778 155.702 0)
@@
 			)
 			(justify left bottom)
+		)
+	)
+	(text "SAO Core4 V2 requires JP5:2-3 closed\nto use GP27 as input for core pulse sense."
+		(exclude_from_sim no)
+		(at 255.524 165.862 0)
+		(effects
+			(font
+				(size 1.27 1.27)
+				(color 194 0 194 1)
+			)
+			(justify left bottom)
